File: project-files/SIO-XS v1p1.brd (EAGLE design)
At the start: 44.2 x 22.6 mm, 11 parts, among them IC1 74HC4066

Commit message: Add files via upload
Parts:
- IC1: value 74HC4066 -> 74HC4066TSSOP-14
Changed lines of the file:
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@@
 </autorouter>
 <elements>
-<element name="CI" library="Consoles Unleashed Eagle Parts Library" package="CIRCLE-1,5X1,5" package3d_urn="urn:adsk.eagle:package:30845/1" value="CI" x="36.195" y="7.62" smashed="yes">
+<element name="CI" library="Consoles Unleashed Eagle Parts Library" package="CIRCLE-1,5X1,5" value="CI" x="36.195" y="7.62" smashed="yes">
 <attribute name="NAME" x="36.195" y="8.636" size="0.8128" layer="25" ratio="7" align="bottom-center"/>
 </element>
-<element name="CE" library="Consoles Unleashed Eagle Parts Library" package="CIRCLE-1,5X1,5" package3d_urn="urn:adsk.eagle:package:30845/1" value="CE" x="38.1" y="9.525" smashed="yes">
+<element name="CE" library="Consoles Unleashed Eagle Parts Library" package="CIRCLE-1,5X1,5" value="CE" x="38.1" y="9.525" smashed="yes">
 <attribute name="NAME" x="38.1" y="10.541" size="0.8128" layer="25" ratio="7" align="bottom-center"/>
 </element>
-<element name="XI" library="Consoles Unleashed Eagle Parts Library" package="CIRCLE-1,5X1,5" package3d_urn="urn:adsk.eagle:package:30845/1" value="XI" x="32.385" y="3.81" smashed="yes">
+<element name="XI" library="Consoles Unleashed Eagle Parts Library" package="CIRCLE-1,5X1,5" value="XI" x="32.385" y="3.81" smashed="yes">
 <attribute name="NAME" x="32.385" y="4.826" size="0.8128" layer="25" ratio="7" align="bottom-center"/>
 </element>
-<element name="XE" library="Consoles Unleashed Eagle Parts Library" package="CIRCLE-1,5X1,5" package3d_urn="urn:adsk.eagle:package:30845/1" value="XE" x="30.48" y="1.905" smashed="yes">
+<element name="XE" library="Consoles Unleashed Eagle Parts Library" package="CIRCLE-1,5X1,5" value="XE" x="30.48" y="1.905" smashed="yes">
 <attribute name="NAME" x="30.48" y="2.921" size="0.8128" layer="25" ratio="7" align="bottom-center"/>
 </element>
@@
 <element name="R4" library="Consoles Unleashed Eagle Parts Library" package="R0805" value="10Kilohm" x="15.24" y="13.081" smashed="yes" rot="R180"/>
 <element name="C1" library="Consoles Unleashed Eagle Parts Library" package="C0805" value="0.1uF" x="23.622" y="13.081" smashed="yes" rot="R180"/>
-<element name="CE1" library="Consoles Unleashed Eagle Parts Library" package="CIRCLE-1,5X1,5" package3d_urn="urn:adsk.eagle:package:30845/1" value="CE" x="34.29" y="5.715" smashed="yes"/>
-<element name="IC1" library="Consoles Unleashed Eagle Parts Library" package="TSSOP-14" value="74HC4066" x="21.59" y="8.89" smashed="yes"/>
+<element name="CE1" library="Consoles Unleashed Eagle Parts Library" package="CIRCLE-1,5X1,5" value="CE" x="34.29" y="5.715" smashed="yes"/>
+<element name="IC1" library="Consoles Unleashed Eagle Parts Library" package="TSSOP-14" value="74HC4066TSSOP-14" x="21.59" y="8.89" smashed="yes"/>
 </elements>
 <signals>
@@
 <via x="6.35" y="15.875" extent="1-16" drill="0.9" diameter="1.4"/>
 <wire x1="8.981" y1="11.781" x2="7.681" y2="13.081" width="0.3048" layer="1"/>
-<wire x1="18.652" y1="7.59" x2="18.652" y2="8.24" width="0.35" layer="1"/>
-<wire x1="18.652" y1="7.59" x2="17.302" y2="7.59" width="0.3048" layer="1"/>
+<wire x1="18.69" y1="7.59" x2="18.69" y2="8.24" width="0.35" layer="1"/>
+<wire x1="18.69" y1="7.59" x2="17.302" y2="7.59" width="0.3048" layer="1"/>
 <wire x1="17.302" y1="7.59" x2="16.129" y2="8.763" width="0.3048" layer="1"/>
 <wire x1="16.129" y1="8.763" x2="16.129" y2="11.303" width="0.3048" layer="1"/>
@@
 <signal name="N$4">
 <via x="39.37" y="15.875" extent="1-16" drill="0.9" diameter="1.4"/>
-<wire x1="24.528" y1="6.94" x2="22.352" y2="6.94" width="0.3048" layer="1"/>
+<wire x1="24.49" y1="6.94" x2="22.352" y2="6.94" width="0.3048" layer="1"/>
 <wire x1="22.352" y1="6.94" x2="22.098" y2="6.686" width="0.3048" layer="1"/>
 <via x="22.098" y="6.686" extent="1-16" drill="0.4" diameter="0.8"/>
@@
 <contactref element="XI" pad="1"/>
 <wire x1="32.385" y1="3.81" x2="31.369" y2="4.826" width="0.8" layer="1"/>
-<wire x1="27.305" y1="8.89" x2="26.179" y2="8.89" width="0.3048" layer="1"/>
-<wire x1="26.179" y1="8.89" x2="24.528" y2="8.89" width="0.3048" layer="1"/>
+<wire x1="27.305" y1="8.89" x2="24.49" y2="8.89" width="0.3048" layer="1"/>
 <via x="27.305" y="8.89" extent="1-16" drill="0.4" diameter="0.8"/>
 <via x="31.369" y="4.826" extent="1-16" drill="0.4" diameter="0.8"/>
@@
 <via x="27.94" y="13.081" extent="1-16" drill="0.4" diameter="0.8"/>
 <wire x1="21.082" y1="11.094" x2="20.828" y2="10.84" width="0.3048" layer="1"/>
-<wire x1="20.828" y1="10.84" x2="18.652" y2="10.84" width="0.3048" layer="1"/>
+<wire x1="20.828" y1="10.84" x2="18.69" y2="10.84" width="0.3048" layer="1"/>
 <wire x1="29.972" y1="16.764" x2="28.448" y2="16.764" width="0.3048" layer="1" curve="70"/>
 <wire x1="29.972" y1="16.764" x2="30.988" y2="16.764" width="0.3048" layer="1" curve="60"/>
@@
 <wire x1="30.48" y1="1.905" x2="29.464" y2="2.921" width="0.8" layer="1"/>
 <wire x1="22.098" y1="10.444" x2="21.844" y2="10.19" width="0.3048" layer="1"/>
-<wire x1="21.844" y1="10.19" x2="18.652" y2="10.19" width="0.3048" layer="1"/>
+<wire x1="21.844" y1="10.19" x2="18.69" y2="10.19" width="0.3048" layer="1"/>
 <wire x1="17.399" y1="11.999" x2="17.399" y2="10.444" width="0.3048" layer="1"/>
 <wire x1="17.399" y1="10.444" x2="17.653" y2="10.19" width="0.3048" layer="1"/>
-<wire x1="17.653" y1="10.19" x2="18.652" y2="10.19" width="0.3048" layer="1"/>
+<wire x1="17.653" y1="10.19" x2="18.69" y2="10.19" width="0.3048" layer="1"/>
 <wire x1="18.481" y1="13.081" x2="17.399" y2="11.999" width="0.3048" layer="1"/>
 <wire x1="22.698003125" y1="10.444" x2="22.200178125" y2="10.669534375" width="0.3048" layer="16"/>
@@
 <wire x1="21.082" y1="7.59" x2="14.194" y2="14.478" width="0.3048" layer="16"/>
 <wire x1="14.194" y1="14.478" x2="10.099" y2="14.478" width="0.3048" layer="16"/>
-<wire x1="24.528" y1="7.59" x2="24.528" y2="8.24" width="0.35" layer="1"/>
-<wire x1="24.528" y1="7.59" x2="21.082" y2="7.59" width="0.3048" layer="1"/>
+<wire x1="24.49" y1="7.59" x2="24.49" y2="8.24" width="0.35" layer="1"/>
+<wire x1="24.49" y1="7.59" x2="21.082" y2="7.59" width="0.3048" layer="1"/>
 <wire x1="36.195" y1="7.62" x2="35.179" y2="8.636" width="0.8" layer="1"/>
-<wire x1="24.528" y1="7.59" x2="30.861" y2="7.59" width="0.3048" layer="1"/>
+<wire x1="24.49" y1="7.59" x2="30.861" y2="7.59" width="0.3048" layer="1"/>
 <via x="30.861" y="7.59" extent="1-16" drill="0.4" diameter="0.8"/>
 <via x="35.179" y="8.636" extent="1-16" drill="0.4" diameter="0.8"/>
@@
 <signal name="N$10">
 <contactref element="R4" pad="1"/>
-<wire x1="24.528" y1="9.54" x2="24.528" y2="10.19" width="0.35" layer="1"/>
+<wire x1="24.49" y1="9.54" x2="24.49" y2="10.19" width="0.35" layer="1"/>
 <wire x1="16.764" y1="12.253" x2="16.764" y2="10.16" width="0.3048" layer="1"/>
 <wire x1="16.764" y1="10.16" x2="17.384" y2="9.54" width="0.3048" layer="1"/>
-<wire x1="17.384" y1="9.54" x2="18.652" y2="9.54" width="0.3048" layer="1"/>
+<wire x1="17.384" y1="9.54" x2="18.69" y2="9.54" width="0.3048" layer="1"/>
 <wire x1="16.764" y1="12.253" x2="16.19" y2="12.827" width="0.3048" layer="1"/>
 <wire x1="16.19" y1="12.827" x2="16.19" y2="13.081" width="0.3048" layer="1"/>
-<wire x1="18.652" y1="9.54" x2="24.528" y2="9.54" width="0.3048" layer="1"/>
+<wire x1="18.69" y1="9.54" x2="24.49" y2="9.54" width="0.3048" layer="1"/>
 <contactref element="IC1" pad="3"/>
 <contactref element="IC1" pad="12"/>
@@
 <vertex x="44.45" y="22.86"/>
 </polygon>
-<wire x1="18.652" y1="8.89" x2="19.939" y2="8.89" width="0.35" layer="1"/>
+<wire x1="18.69" y1="8.89" x2="19.939" y2="8.89" width="0.35" layer="1"/>
 <wire x1="19.939" y1="8.89" x2="20.193" y2="8.636" width="0.35" layer="1"/>
 <wire x1="20.193" y1="8.636" x2="20.193" y2="7.211" width="0.35" layer="1"/>
 <wire x1="20.193" y1="7.211" x2="19.922" y2="6.94" width="0.35" layer="1"/>
-<wire x1="19.922" y1="6.94" x2="18.652" y2="6.94" width="0.35" layer="1"/>
-<wire x1="18.652" y1="6.94" x2="17.145" y2="6.94" width="0.35" layer="1"/>
+<wire x1="19.922" y1="6.94" x2="18.69" y2="6.94" width="0.35" layer="1"/>
+<wire x1="18.69" y1="6.94" x2="17.145" y2="6.94" width="0.35" layer="1"/>
 <wire x1="43.18" y1="20.32" x2="43.18" y2="21.59" width="0.4064" layer="1"/>
 <wire x1="43.18" y1="19.05" x2="43.18" y2="17.78" width="0.4064" layer="1"/>
@@
 <wire x1="1.27" y1="19.685" x2="1.27" y2="18.415" width="0.4064" layer="1"/>
 <wire x1="1.27" y1="15.875" x2="1.27" y2="17.145" width="0.4064" layer="1"/>
-<wire x1="18.652" y1="8.89" x2="17.145" y2="8.89" width="0.35" layer="1"/>
+<wire x1="18.69" y1="8.89" x2="17.145" y2="8.89" width="0.35" layer="1"/>
 </signal>
 <signal name="+3.3V">
@@
 <wire x1="23.323" y1="10.84" x2="22.672" y2="11.491" width="0.35" layer="1"/>
 <wire x1="22.672" y1="13.081" x2="22.672" y2="11.491" width="0.35" layer="1"/>
-<wire x1="23.323" y1="10.84" x2="24.528" y2="10.84" width="0.35" layer="1"/>
+<wire x1="23.323" y1="10.84" x2="24.49" y2="10.84" width="0.35" layer="1"/>
 <wire x1="22.672" y1="13.081" x2="20.381" y2="13.081" width="0.4064" layer="1"/>
 <wire x1="21.59" y1="18.334996875" x2="22.01095625" y2="19.53765" width="0.508" layer="1" curve="-30"/>
@@
 which will not be processed correctly with this version.
 </note>
-<note version="8.3" severity="warning">
-Since Version 8.3, EAGLE supports URNs for individual library
-assets (packages, symbols, and devices). The URNs of those assets
-will not be understood (or retained) with this version.
-</note>
-<note version="8.3" severity="warning">
-Since Version 8.3, EAGLE supports the association of 3D packages
-with devices in libraries, schematics, and board files. Those 3D
-packages will not be understood (or retained) with this version.
-</note>
 </compatibility>
