File: project-files/SIO-XS v1p1.sch (EAGLE design)
At the start: 11 parts, among them IC1 74HC4066

Commit message: Add files via upload
Parts:
- IC1: value 74HC4066 -> 74HC4066TSSOP-14; device Consoles Unleashed Eagle Parts Library:74HC4066 -> Consoles Unleashed Eagle Parts Library:74HC4066TSSOP-14
Changed lines of the file:
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@@
 </classes>
 <parts>
-<part name="CI" library="Consoles Unleashed Eagle Parts Library" deviceset="PADS" device="CIRCLE-1,5X1,5" package3d_urn="urn:adsk.eagle:package:30845/1" value="CI"/>
-<part name="CE" library="Consoles Unleashed Eagle Parts Library" deviceset="PADS" device="CIRCLE-1,5X1,5" package3d_urn="urn:adsk.eagle:package:30845/1" value="CE"/>
-<part name="XI" library="Consoles Unleashed Eagle Parts Library" deviceset="PADS" device="CIRCLE-1,5X1,5" package3d_urn="urn:adsk.eagle:package:30845/1" value="XI"/>
-<part name="XE" library="Consoles Unleashed Eagle Parts Library" deviceset="PADS" device="CIRCLE-1,5X1,5" package3d_urn="urn:adsk.eagle:package:30845/1" value="XE"/>
+<part name="CI" library="Consoles Unleashed Eagle Parts Library" deviceset="PADS" device="CIRCLE-1,5X1,5" value="CI"/>
+<part name="CE" library="Consoles Unleashed Eagle Parts Library" deviceset="PADS" device="CIRCLE-1,5X1,5" value="CE"/>
+<part name="XI" library="Consoles Unleashed Eagle Parts Library" deviceset="PADS" device="CIRCLE-1,5X1,5" value="XI"/>
+<part name="XE" library="Consoles Unleashed Eagle Parts Library" deviceset="PADS" device="CIRCLE-1,5X1,5" value="XE"/>
 <part name="R1" library="Consoles Unleashed Eagle Parts Library" deviceset="RESISTORS" device="R0805" value="47Kilohm"/>
 <part name="R2" library="Consoles Unleashed Eagle Parts Library" deviceset="RESISTORS" device="R0805" value="10Kilohm"/>
@@
 <part name="+3V1" library="Consoles Unleashed Eagle Parts Library" deviceset="+3V3" device=""/>
 <part name="GND1" library="Consoles Unleashed Eagle Parts Library" deviceset="GND" device=""/>
-<part name="CE1" library="Consoles Unleashed Eagle Parts Library" deviceset="PADS" device="CIRCLE-1,5X1,5" package3d_urn="urn:adsk.eagle:package:30845/1" value="CE"/>
-<part name="IC1" library="Consoles Unleashed Eagle Parts Library" deviceset="74HC4066" device=""/>
+<part name="CE1" library="Consoles Unleashed Eagle Parts Library" deviceset="PADS" device="CIRCLE-1,5X1,5" value="CE"/>
+<part name="IC1" library="Consoles Unleashed Eagle Parts Library" deviceset="74HC4066" device="TSSOP-14"/>
 </parts>
 <sheets>
@@
 will not be understood (or retained) with this version.
 </note>
-<note version="8.3" severity="warning">
-Since Version 8.3, EAGLE supports the association of 3D packages
-with devices in libraries, schematics, and board files. Those 3D
-packages will not be understood (or retained) with this version.
-</note>
 </compatibility>
